Commit message: Phase 2: Optimized Pick-and-Place for Sim2Real. Restored grasp stability with weight tuning and raised transport threshold to 3cm. Includes updated DEPLOYMENT_MANIFEST.md.

File: src/isaac_so_arm101/robots/trs_so100/urdf/so_arm100.urdf (robot description, URDF)
Before this commit: robot so_arm100, 7 links, 6 joints
Links:
- link gripper: geometry collision mesh filename=assets/Fixed_Jaw.stl; visual mesh filename=assets/Fixed_Jaw.stl
- link jaw: geometry collision mesh filename=assets/Moving_Jaw.stl; visual mesh filename=assets/Moving_Jaw.stl
- link lower_arm: geometry collision box size=0.045 0.045 0.14; visual mesh filename=assets/Lower_Arm.stl
- link shoulder: geometry collision box size=0.06 0.11 0.06; visual mesh filename=assets/Rotation_Pitch.stl
- link upper_arm: geometry collision box size=0.045 0.14 0.045; visual mesh filename=assets/Upper_Arm.stl
- link wrist: geometry collision box size=0.035 0.06 0.035; visual mesh filename=assets/Wrist_Pitch_Roll.stl
Joints:
- joint gripper: limit lower=-0.2 upper=2.0 effort=35 velocity=1 -> lower=0.0 upper=1.2 effort=35 velocity=1
- joint shoulder_pan: limit lower=-2 upper=2 effort=35 velocity=1 -> lower=-3.1 upper=3.1 effort=35 velocity=1
